File: Eagle/DIY-Cellphone.sch (EAGLE design)
At the start: 39 parts, among them IC1 MEGA1284, J1 ISP, U1 MCP73831, U7 M10_HDWITHOUT_EXCLUSION, X1 BU-SMA-V, X3 CCM03-3002 R102

Commit message: Update silk screen labels, polygon isolate, etc.
Parts:
- renumbered JP6 to MIC, RESET to RST, U$5 to SPEAKER
Connections:
- net COL1 renamed PA5
- net COL2 renamed PA7
- net COL3 renamed PC7
- net LCD_D/C renamed PD6
- net LCD_DN renamed PD7
- net LCD_LED renamed PC1
- net LCD_RST renamed PD5
- net LCD_SCE renamed PD4
- net LCD_SCLK renamed PC0
- net N$2 renamed PC6
- net N$3 renamed PC5
- net N$4 renamed PC4
- net ROW1 renamed PA6
- net ROW2 renamed PA4
- net ROW3 renamed PA3
- net ROW4 renamed PA2
- net ROW5 renamed PA1
- net ROW6 renamed PA0
- new net PC2: IC1.(TCK/PCINT18)PC2
Changed lines of the file:
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@@
 <part name="C15" library="cellphone-rcl" deviceset="C-EU" device="C1206" value="18pF"/>
 <part name="C16" library="cellphone-rcl" deviceset="CPOL-US" device="D/7343-31R" value="1000uF"/>
-<part name="U$5" library="cellphone" deviceset="MINI-SIREN" device=""/>
-<part name="RESET" library="cellphone" deviceset="BUTTON-2" device="" value="BUTTON"/>
+<part name="SPEAKER" library="cellphone" deviceset="MINI-SIREN" device=""/>
+<part name="RST" library="cellphone" deviceset="BUTTON-2" device="" value="BUTTON"/>
 <part name="R9" library="cellphone-rcl" deviceset="R-US_" device="R1206" value="470"/>
 <part name="LED1" library="cellphone-led" deviceset="LED" device="SMT1206"/>
 <part name="LED2" library="cellphone-led" deviceset="LED" device="SMT1206"/>
 <part name="R10" library="cellphone-rcl" deviceset="R-US_" device="R1206" value="470"/>
-<part name="JP6" library="pinhead" deviceset="PINHD-1X2" device=""/>
+<part name="MIC" library="pinhead" deviceset="PINHD-1X2" device=""/>
 <part name="JP2" library="pinhead" deviceset="PINHD-1X8" device=""/>
 <part name="JP5" library="pinhead" deviceset="PINHD-1X4" device=""/>
@@
 <instance part="C15" gate="G$1" x="-63.5" y="101.6" rot="R270"/>
 <instance part="C16" gate="G$1" x="302.26" y="213.36"/>
-<instance part="U$5" gate="G$1" x="149.86" y="233.68" rot="R270"/>
-<instance part="RESET" gate="G$1" x="-66.04" y="109.22"/>
+<instance part="SPEAKER" gate="G$1" x="149.86" y="233.68" rot="R270"/>
+<instance part="RST" gate="G$1" x="-66.04" y="109.22"/>
 <instance part="R9" gate="G$1" x="292.1" y="254" rot="R90"/>
 <instance part="LED1" gate="G$1" x="292.1" y="266.7"/>
 <instance part="LED2" gate="G$1" x="162.56" y="175.26" rot="R90"/>
 <instance part="R10" gate="G$1" x="177.8" y="175.26"/>
-<instance part="JP6" gate="G$1" x="165.1" y="251.46" rot="R270"/>
+<instance part="MIC" gate="G$1" x="165.1" y="251.46" rot="R270"/>
 <instance part="JP2" gate="A" x="50.8" y="99.06"/>
 <instance part="JP5" gate="A" x="50.8" y="25.4"/>
@@
 <label x="-78.74" y="91.44" size="1.778" layer="95"/>
 <wire x1="-76.2" y1="109.22" x2="-71.12" y2="109.22" width="0.1524" layer="91"/>
-<pinref part="RESET" gate="G$1" pin="P"/>
+<pinref part="RST" gate="G$1" pin="P"/>
 </segment>
 <segment>
@@
 <wire x1="116.84" y1="233.68" x2="144.78" y2="233.68" width="0.1524" layer="91"/>
 <wire x1="144.78" y1="233.68" x2="144.78" y2="238.76" width="0.1524" layer="91"/>
-<pinref part="U$5" gate="G$1" pin="1"/>
+<pinref part="SPEAKER" gate="G$1" pin="1"/>
 <wire x1="144.78" y1="238.76" x2="149.86" y2="238.76" width="0.1524" layer="91"/>
 </segment>
@@
 <label x="137.16" y="231.14" size="1.778" layer="95"/>
 <wire x1="116.84" y1="231.14" x2="142.24" y2="231.14" width="0.1524" layer="91"/>
-<pinref part="U$5" gate="G$1" pin="2"/>
+<pinref part="SPEAKER" gate="G$1" pin="2"/>
 <wire x1="149.86" y1="228.6" x2="142.24" y2="228.6" width="0.1524" layer="91"/>
 <wire x1="142.24" y1="228.6" x2="142.24" y2="231.14" width="0.1524" layer="91"/>
@@
 <wire x1="157.48" y1="246.38" x2="157.48" y2="284.48" width="0.1524" layer="91"/>
 <label x="157.48" y="276.86" size="1.778" layer="95" rot="R90"/>
-<pinref part="JP6" gate="G$1" pin="2"/>
+<pinref part="MIC" gate="G$1" pin="2"/>
 <wire x1="165.1" y1="246.38" x2="165.1" y2="254" width="0.1524" layer="91"/>
 </segment>
@@
 <wire x1="175.26" y1="246.38" x2="175.26" y2="284.48" width="0.1524" layer="91"/>
 <label x="175.26" y="276.86" size="1.778" layer="95" rot="R90"/>
-<pinref part="JP6" gate="G$1" pin="1"/>
+<pinref part="MIC" gate="G$1" pin="1"/>
 <wire x1="167.64" y1="246.38" x2="167.64" y2="254" width="0.1524" layer="91"/>
 </segment>
@@
 <wire x1="-55.88" y1="109.22" x2="-60.96" y2="109.22" width="0.1524" layer="91"/>
 <junction x="-55.88" y="109.22"/>
-<pinref part="RESET" gate="G$1" pin="S"/>
+<pinref part="RST" gate="G$1" pin="S"/>
 </segment>
 <segment>
@@
 </segment>
 </net>
-<net name="ROW6" class="0">
+<net name="PA0" class="0">
 <segment>
 <pinref part="IC1" gate="G$1" pin="(ADC0/PCINT0)PA0"/>
@@
 </segment>
 </net>
-<net name="ROW5" class="0">
+<net name="PA1" class="0">
 <segment>
 <pinref part="IC1" gate="G$1" pin="(ADC1/PCINT1)PA1"/>
@@
 </segment>
 </net>
-<net name="ROW4" class="0">
+<net name="PA2" class="0">
 <segment>
 <pinref part="IC1" gate="G$1" pin="(ADC2/PCINT2)PA2"/>
@@
 </segment>
 </net>
-<net name="ROW3" class="0">
+<net name="PA3" class="0">
 <segment>
 <pinref part="IC1" gate="G$1" pin="(ADC3/PCINT3)PA3"/>
@@
 </segment>
 </net>
-<net name="COL1" class="0">
+<net name="PA5" class="0">
 <segment>
 <pinref part="IC1" gate="G$1" pin="(ADC5/PCINT5)PA5"/>
@@
 </segment>
 </net>
-<net name="COL2" class="0">
+<net name="PA7" class="0">
 <segment>
 <pinref part="IC1" gate="G$1" pin="(ADC7/PCINT7)PA7"/>
@@
 </segment>
 </net>
-<net name="COL3" class="0">
+<net name="PC7" class="0">
 <segment>
 <pinref part="IC1" gate="G$1" pin="(TOSC2/PCINT23)PC7"/>
@@
 </segment>
 </net>
-<net name="ROW2" class="0">
+<net name="PA4" class="0">
 <segment>
 <pinref part="IC1" gate="G$1" pin="(ADC4/PCINT4)PA4"/>
@@
 </segment>
 </net>
-<net name="ROW1" class="0">
+<net name="PA6" class="0">
 <segment>
 <pinref part="IC1" gate="G$1" pin="(ADC6/PCINT6)PA6"/>
@@
 </segment>
 </net>
-<net name="LCD_SCE" class="0">
+<net name="PD4" class="0">
 <segment>
 <pinref part="IC1" gate="G$1" pin="(XCK1/OC1B/PCINT28)PD4"/>
@@
 </segment>
 </net>
-<net name="LCD_RST" class="0">
+<net name="PD5" class="0">
 <segment>
 <pinref part="IC1" gate="G$1" pin="(OC1A/PCINT29)PD5"/>
@@
 </segment>
 </net>
-<net name="LCD_D/C" class="0">
+<net name="PD6" class="0">
 <segment>
 <pinref part="IC1" gate="G$1" pin="(OC2B/ICP/PCINT30)PD6"/>
@@
 </segment>
 </net>
-<net name="LCD_DN" class="0">
+<net name="PD7" class="0">
 <segment>
 <pinref part="IC1" gate="G$1" pin="(OC2A/PCINT31)PD7"/>
@@
 </segment>
 </net>
-<net name="LCD_SCLK" class="0">
+<net name="PC0" class="0">
 <segment>
 <pinref part="IC1" gate="G$1" pin="(SCL/PCINT16)PC0"/>
@@
 </segment>
 </net>
-<net name="LCD_LED" class="0">
+<net name="PC1" class="0">
 <segment>
 <pinref part="IC1" gate="G$1" pin="(SDA/PCINT17)PC1"/>
@@
 </segment>
 </net>
-<net name="N$2" class="0">
+<net name="PC6" class="0">
 <segment>
 <pinref part="IC1" gate="G$1" pin="(TOSC1/PCINT22)PC6"/>
 <wire x1="5.08" y1="48.26" x2="48.26" y2="48.26" width="0.1524" layer="91"/>
 <pinref part="JP1" gate="A" pin="3"/>
-</segment>
-</net>
-<net name="N$3" class="0">
+<label x="12.7" y="48.26" size="1.778" layer="95"/>
+</segment>
+</net>
+<net name="PC5" class="0">
 <segment>
 <pinref part="IC1" gate="G$1" pin="(TDI/PCINT21)PC5"/>
 <wire x1="5.08" y1="50.8" x2="48.26" y2="50.8" width="0.1524" layer="91"/>
 <pinref part="JP1" gate="A" pin="2"/>
-</segment>
-</net>
-<net name="N$4" class="0">
+<label x="12.7" y="50.8" size="1.778" layer="95"/>
+</segment>
+</net>
+<net name="PC4" class="0">
 <segment>
 <pinref part="IC1" gate="G$1" pin="(TDO/PCINT20)PC4"/>
 <wire x1="5.08" y1="53.34" x2="48.26" y2="53.34" width="0.1524" layer="91"/>
 <pinref part="JP1" gate="A" pin="1"/>
-</segment>
-</net>
+<label x="12.7" y="53.34" size="1.778" layer="95"/>
+</segment>
+</net>
+<net name="PC2" class="0">
+<segment>
+<pinref part="IC1" gate="G$1" pin="(TCK/PCINT18)PC2"/>
+<wire x1="5.08" y1="58.42" x2="50.8" y2="58.42" width="0.1524" layer="91"/>
+<label x="12.7" y="58.42" size="1.778" layer="95"/>
+</segment>
+</net>

Commit message: Break out I2C and SPI pins.
Parts:
- added JP4, JP6: (no value), pinhead:PINHD-1X3
Connections:
- net MISO: now also JP6.2
- net MOSI: now also JP6.1
- net PC0: now also JP4.1
- net PC1: now also JP4.2
- net PC2: now also JP4.3
- net SCK: now also JP6.3
Changed lines of the file:
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@@
 <part name="JP1" library="pinhead" deviceset="PINHD-1X4" device=""/>
 <part name="JP7" library="cellphone" deviceset="ARDUINO_SERIAL_PROGRAM" device="SMD-NOHOLES"/>
+<part name="JP4" library="pinhead" deviceset="PINHD-1X3" device=""/>
+<part name="JP6" library="pinhead" deviceset="PINHD-1X3" device=""/>
 </parts>
 <sheets>
@@
 <instance part="JP1" gate="A" x="50.8" y="48.26"/>
 <instance part="JP7" gate="G$1" x="-35.56" y="-10.16"/>
+<instance part="JP4" gate="A" x="50.8" y="60.96"/>
+<instance part="JP6" gate="A" x="50.8" y="71.12"/>
 </instances>
 <busses>
@@
 <segment>
 <pinref part="IC1" gate="G$1" pin="(SCK/PCINT15)PB7"/>
-<wire x1="5.08" y1="68.58" x2="17.78" y2="68.58" width="0.1524" layer="91"/>
+<wire x1="5.08" y1="68.58" x2="48.26" y2="68.58" width="0.1524" layer="91"/>
 <label x="12.7" y="68.58" size="1.778" layer="95"/>
+<pinref part="JP6" gate="A" pin="3"/>
 </segment>
 <segment>
@@
 <segment>
 <pinref part="IC1" gate="G$1" pin="(MISO/PCINT14)PB6"/>
-<wire x1="5.08" y1="71.12" x2="17.78" y2="71.12" width="0.1524" layer="91"/>
+<wire x1="5.08" y1="71.12" x2="48.26" y2="71.12" width="0.1524" layer="91"/>
 <label x="12.7" y="71.12" size="1.778" layer="95"/>
+<pinref part="JP6" gate="A" pin="2"/>
 </segment>
 <segment>
@@
 <segment>
 <pinref part="IC1" gate="G$1" pin="(MOSI/PCINT13)PB5"/>
-<wire x1="5.08" y1="73.66" x2="17.78" y2="73.66" width="0.1524" layer="91"/>
+<wire x1="5.08" y1="73.66" x2="48.26" y2="73.66" width="0.1524" layer="91"/>
 <label x="12.7" y="73.66" size="1.778" layer="95"/>
+<pinref part="JP6" gate="A" pin="1"/>
 </segment>
 <segment>
@@
 <pinref part="IC1" gate="G$1" pin="(SCL/PCINT16)PC0"/>
 <label x="12.7" y="63.5" size="1.778" layer="95"/>
-<wire x1="5.08" y1="63.5" x2="27.94" y2="63.5" width="0.1524" layer="91"/>
-<wire x1="27.94" y1="63.5" x2="50.8" y2="63.5" width="0.1524" layer="91"/>
+<wire x1="5.08" y1="63.5" x2="48.26" y2="63.5" width="0.1524" layer="91"/>
+<pinref part="JP4" gate="A" pin="1"/>
 </segment>
 </net>
@@
 <pinref part="IC1" gate="G$1" pin="(SDA/PCINT17)PC1"/>
 <label x="12.7" y="60.96" size="1.778" layer="95"/>
-<wire x1="5.08" y1="60.96" x2="25.4" y2="60.96" width="0.1524" layer="91"/>
-<wire x1="25.4" y1="60.96" x2="50.8" y2="60.96" width="0.1524" layer="91"/>
+<wire x1="5.08" y1="60.96" x2="48.26" y2="60.96" width="0.1524" layer="91"/>
+<pinref part="JP4" gate="A" pin="2"/>
 </segment>
 </net>
@@
 <segment>
 <pinref part="IC1" gate="G$1" pin="(TCK/PCINT18)PC2"/>
-<wire x1="5.08" y1="58.42" x2="50.8" y2="58.42" width="0.1524" layer="91"/>
+<wire x1="5.08" y1="58.42" x2="48.26" y2="58.42" width="0.1524" layer="91"/>
 <label x="12.7" y="58.42" size="1.778" layer="95"/>
-</segment>
-</net>
+<pinref part="JP4" gate="A" pin="3"/>
+</segment>
+</net>

Commit message: Break out power and ground.
Parts:
- added JP8, JP9: (no value), pinhead:PINHD-1X2
Connections:
- net GND: now also JP8.2, JP9.2
- net VCC: now also JP8.1, JP9.1
Changed lines of the file:
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@@
 <part name="JP4" library="pinhead" deviceset="PINHD-1X3" device=""/>
 <part name="JP6" library="pinhead" deviceset="PINHD-1X3" device=""/>
+<part name="JP8" library="pinhead" deviceset="PINHD-1X2" device=""/>
+<part name="JP9" library="pinhead" deviceset="PINHD-1X2" device=""/>
 </parts>
 <sheets>
@@
 <instance part="JP4" gate="A" x="50.8" y="60.96"/>
 <instance part="JP6" gate="A" x="50.8" y="71.12"/>
+<instance part="JP8" gate="G$1" x="50.8" y="137.16"/>
+<instance part="JP9" gate="G$1" x="50.8" y="124.46"/>
 </instances>
 <busses>
@@
 <pinref part="U1" gate="G$1" pin="VBAT"/>
 <pinref part="C4" gate="G$1" pin="1"/>
+</segment>
+<segment>
+<pinref part="JP8" gate="G$1" pin="1"/>
+<wire x1="48.26" y1="139.7" x2="30.48" y2="139.7" width="0.1524" layer="91"/>
+<label x="30.48" y="139.7" size="1.778" layer="95"/>
+</segment>
+<segment>
+<pinref part="JP9" gate="G$1" pin="1"/>
+<wire x1="48.26" y1="127" x2="30.48" y2="127" width="0.1524" layer="91"/>
+<label x="30.48" y="127" size="1.778" layer="95"/>
 </segment>
 </net>
@@
 <label x="195.58" y="172.72" size="1.778" layer="95" rot="R90"/>
 </segment>
+<segment>
+<pinref part="JP8" gate="G$1" pin="2"/>
+<wire x1="48.26" y1="137.16" x2="30.48" y2="137.16" width="0.1524" layer="91"/>
+<label x="30.48" y="137.16" size="1.778" layer="95"/>
+</segment>
+<segment>
+<pinref part="JP9" gate="G$1" pin="2"/>
+<wire x1="48.26" y1="124.46" x2="30.48" y2="124.46" width="0.1524" layer="91"/>
+<label x="30.48" y="124.46" size="1.778" layer="95"/>
+</segment>
 </net>

Commit message: Add LEDs for power and pin 13.
Parts:
- added LED3: PWR, cellphone-led:LEDSMT1206
- added LED4: 13, cellphone-led:LEDSMT1206
- added R1, R5: 470, cellphone-rcl:R-US_R1206
Connections:
- new net N$2: LED3.C, R1.2
- new net N$3: LED4.C, R5.2
- net GND: now also R1.1, R5.1
- net PD5: now also LED4.A
- net VCC: now also LED3.A
Changed lines of the file:
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@@
 <part name="JP8" library="pinhead" deviceset="PINHD-1X2" device=""/>
 <part name="JP9" library="pinhead" deviceset="PINHD-1X2" device=""/>
+<part name="LED3" library="cellphone-led" deviceset="LED" device="SMT1206" value="PWR"/>
+<part name="R1" library="cellphone-rcl" deviceset="R-US_" device="R1206" value="470"/>
+<part name="LED4" library="cellphone-led" deviceset="LED" device="SMT1206" value="13"/>
+<part name="R5" library="cellphone-rcl" deviceset="R-US_" device="R1206" value="470"/>
 </parts>
 <sheets>
@@
 <instance part="JP8" gate="G$1" x="50.8" y="137.16"/>
 <instance part="JP9" gate="G$1" x="50.8" y="124.46"/>
+<instance part="LED3" gate="G$1" x="266.7" y="213.36"/>
+<instance part="R1" gate="G$1" x="266.7" y="203.2" rot="R90"/>
+<instance part="LED4" gate="G$1" x="58.42" y="17.78"/>
+<instance part="R5" gate="G$1" x="58.42" y="5.08" rot="R90"/>
 </instances>
 <busses>
@@
 <pinref part="C16" gate="G$1" pin="+"/>
 <junction x="302.26" y="215.9"/>
+<pinref part="LED3" gate="G$1" pin="A"/>
+<wire x1="289.56" y1="215.9" x2="266.7" y2="215.9" width="0.1524" layer="91"/>
+<junction x="289.56" y="215.9"/>
 </segment>
 <segment>
@@
 <wire x1="302.26" y1="208.28" x2="289.56" y2="208.28" width="0.1524" layer="91"/>
 <junction x="302.26" y="208.28"/>
+<wire x1="289.56" y1="208.28" x2="274.32" y2="208.28" width="0.1524" layer="91"/>
+<wire x1="274.32" y1="208.28" x2="274.32" y2="198.12" width="0.1524" layer="91"/>
+<junction x="289.56" y="208.28"/>
+<pinref part="R1" gate="G$1" pin="1"/>
+<wire x1="274.32" y1="198.12" x2="266.7" y2="198.12" width="0.1524" layer="91"/>
 </segment>
 <segment>
@@
 <wire x1="48.26" y1="124.46" x2="30.48" y2="124.46" width="0.1524" layer="91"/>
 <label x="30.48" y="124.46" size="1.778" layer="95"/>
+</segment>
+<segment>
+<pinref part="R5" gate="G$1" pin="1"/>
+<wire x1="58.42" y1="0" x2="58.42" y2="-5.08" width="0.1524" layer="91"/>
+<label x="55.88" y="-7.62" size="1.778" layer="95"/>
 </segment>
 </net>
@@
 <label x="12.7" y="27.94" size="1.778" layer="95"/>
 <pinref part="JP5" gate="A" pin="2"/>
+<pinref part="LED4" gate="G$1" pin="A"/>
+<wire x1="48.26" y1="27.94" x2="58.42" y2="27.94" width="0.1524" layer="91"/>
+<wire x1="58.42" y1="27.94" x2="58.42" y2="20.32" width="0.1524" layer="91"/>
+<junction x="48.26" y="27.94"/>
 </segment>
 </net>
@@
 </segment>
 </net>
+<net name="N$2" class="0">
+<segment>
+<pinref part="LED3" gate="G$1" pin="C"/>
+<pinref part="R1" gate="G$1" pin="2"/>
+</segment>
+</net>
+<net name="N$3" class="0">
+<segment>
+<pinref part="LED4" gate="G$1" pin="C"/>
+<pinref part="R5" gate="G$1" pin="2"/>
+<wire x1="58.42" y1="12.7" x2="58.42" y2="10.16" width="0.1524" layer="91"/>
+</segment>
+</net>
